Commit message: Fix urdf

File: src/car_description/urdf/five_link_car.urdf.xacro (robot description, xacro)
@@ -22,5 +22,5 @@
     <link name="link5">
       <visual name="">
-        <origin xyz="${link_width} 0.0 0.0" rpy="0.0 0.0 0.0"/>
+        <origin xyz="0 0.0 0.0" rpy="0.0 0.0 0.0"/>
         <geometry>
           <box size="${link_width} ${link5_length} ${link_width}"/>
@@ -31,16 +31,15 @@
       </visual>
       <collision>
-        <origin xyz="${link_width} 0.0 0.0" rpy="0.0 0.0 0.0"/>
+        <origin xyz="0 0.0 0.0" rpy="0.0 0.0 0.0"/>
         <geometry>
           <box size="${link_width} ${link5_length} ${link_width}"/>
         </geometry>
       </collision>
-      <xacro:Box_Inertial_Matrix m="${mass_val}" l="${link_width}" w="${link5_length}" h="${link_width}" x_offset="${link_width}" y_offset="0.0" z_offset="0.0" />
+      <xacro:Box_Inertial_Matrix m="${mass_val}" l="${link_width}" w="${link5_length}" h="${link_width}" x_offset="0" y_offset="0.0" z_offset="0.0" />
     </link>
-    <joint name="link5_joint" type="revolute">
-      <origin xyz="${x_offset} ${y_offset} ${z_offset - link_width / 2}" rpy="0.0 0.0 0.0"/>
+    <joint name="link5_joint" type="fixed">
+      <origin xyz="${link_width} ${y_offset} ${z_offset - link_width / 2}" rpy="0.0 0.0 0.0"/>
       <parent link="${connected_to}"/>
       <child link="link5"/>
-      <limit lower="0.0" upper="0.0" effort="0.0" velocity="0.0"/>
     </joint>
     <link name="link1">
@@ -63,5 +62,5 @@
     </link>
     <joint name="link1_joint" type="continuous">
-      <origin xyz="${link_width/2} ${link5_length / 2} 0.0" rpy="0.0 0.0 0.0"/>
+      <origin xyz="${-link_width/2} ${link5_length / 2} 0.0" rpy="0.0 0.0 0.0"/>
       <parent link="link5"/>
       <child link="link1"/>
@@ -111,6 +110,6 @@
     </link>
     <joint name="link3_joint" type="continuous">
-      <origin xyz="0 ${link2_length} 0.0" rpy="${-0.6435*2} 0.0 0.0"/>
-      <parent link="link2"/>
+      <origin xyz="0 ${-link4_length} 0.0" rpy="${-0.6435} 0.0 0.0"/>
+      <parent link="link4"/>
       <child link="link3"/>
       <axis xyz="1 0.0 0.0"/>
@@ -118,5 +117,5 @@
     <link name="link4">
       <visual name="">
-        <origin xyz="${-link_width/2} ${link4_length /2} 0.0" rpy="0.0 0.0 0.0"/>
+        <origin xyz="${-link_width/2} ${-link4_length /2} 0.0" rpy="0.0 0.0 0.0"/>
         <geometry>
           <box size="${link_width} ${link4_length} ${link_width}"/>
@@ -127,14 +126,14 @@
       </visual>
       <collision>
-        <origin xyz="${-link_width/2} ${link4_length /2} 0.0" rpy="0 0.0 0.0"/>
+        <origin xyz="${-link_width/2} ${-link4_length /2} 0.0" rpy="0 0.0 0.0"/>
         <geometry>
           <box size="${link_width} ${link4_length} ${link_width}"/>
         </geometry>
       </collision>
-      <xacro:Box_Inertial_Matrix m="${mass_val}" l="${link_width}" w="${link4_length}" h="${link_width}" x_offset="${-link_width/2}" y_offset="${link4_length/2}" z_offset="0.0" />
+      <xacro:Box_Inertial_Matrix m="${mass_val}" l="${link_width}" w="${link4_length}" h="${link_width}" x_offset="${-link_width/2}" y_offset="${-link4_length/2}" z_offset="0.0" />
     </link>
     <joint name="link4_joint" type="continuous">
-      <origin xyz="0 ${link3_length} 0.0" rpy="${pi+0.6435} 0.0 0.0"/>
-      <parent link="link3"/>
+      <origin xyz="${-link_width/2} ${-link5_length/2} 0.0" rpy="0 0.0 0.0"/>
+      <parent link="link5"/>
       <child link="link4"/>
       <axis xyz="1 0 0.0"/>
@@ -160,6 +159,7 @@
       </geometry>
     </collision>
+    <xacro:Box_Inertial_Matrix m="${mass_val}" l="${base_link_length}" w="${base_link_length}" h="${base_link_height}" x_offset="0.0" y_offset="0.0" z_offset="${base_link_height / 2}" />
   </link>
-  <joint name="world_to_base" type="fixed">
+  <joint name="base_world" type="fixed">
     <parent link="world"/>
     <child link="base_link"/>
@@ -167,11 +167,11 @@
   <xacro:five_link_struct connected_to="base_link" x_offset="0" y_offset="0.0" z_offset="${base_link_height}"/>
   <gazebo>
-    <joint name="link4_conn_link5" type="revolute">
-      <parent>link4</parent>
-      <child>link5</child>
+    <joint name="link3_conn_link2" type="revolute">
+      <parent>link2</parent>
+      <child>link3</child>
       <axis>
           <xyz>1 0 0</xyz>
       </axis>
-      <pose>${link_width/2} ${-link5_length/2} 0 0 0 0</pose>
+      <pose>0 ${link3_length} 0 0 0 0</pose>
       <limit lower="-3.14" upper="3.14" effort="10" velocity="10"/>
     </joint>

Commit message: Add limit

File: src/car_description/urdf/five_link_car.urdf.xacro (robot description, xacro)
@@ -61,9 +61,10 @@
       <xacro:Box_Inertial_Matrix m="${mass_val}" l="${link_width}" w="${link1_length}" h="${link_width}" x_offset="${-link_width/2}" y_offset="${link1_length/2}" z_offset="0.0" />
     </link>
-    <joint name="link1_joint" type="continuous">
+    <joint name="link1_joint" type="revolute">
       <origin xyz="${-link_width/2} ${link5_length / 2} 0.0" rpy="0.0 0.0 0.0"/>
       <parent link="link5"/>
       <child link="link1"/>
       <axis xyz="1 0 0.0"/>
+      <limit lower="-1.74" upper="0.44" effort="0.0" velocity="0.0"/>
     </joint>
     <link name="link2">
@@ -85,9 +86,10 @@
       <xacro:Box_Inertial_Matrix m="${mass_val}" l="${link_width}" w="${link2_length}" h="${link_width}" x_offset="${link_width/2}" y_offset="${link2_length/2}" z_offset="0.0" />
     </link>
-    <joint name="link2_joint" type="continuous">
+    <joint name="link2_joint" type="revolute">
       <origin xyz="0 ${link1_length} 0.0" rpy="${-pi+0.6435} 0.0 0.0"/>
       <parent link="link1"/>
       <child link="link2"/>
       <axis xyz="1 0.0 0.0"/>
+      <limit lower="-0.4" upper="2.5" effort="0.0" velocity="0.0"/>
     </joint>
     <link name="link3">
@@ -109,9 +111,10 @@
       <xacro:Box_Inertial_Matrix m="${mass_val}" l="${link_width}" w="${link3_length}" h="${link_width}" x_offset="${link_width/2}" y_offset="${link3_length/2}" z_offset="0.0" />
     </link>
-    <joint name="link3_joint" type="continuous">
+    <joint name="link3_joint" type="revolute">
       <origin xyz="0 ${-link4_length} 0.0" rpy="${-0.6435} 0.0 0.0"/>
       <parent link="link4"/>
       <child link="link3"/>
       <axis xyz="1 0.0 0.0"/>
+      <limit lower="-2.5" upper="0.4" effort="0.0" velocity="0.0"/>
     </joint>
     <link name="link4">
@@ -133,9 +136,10 @@
       <xacro:Box_Inertial_Matrix m="${mass_val}" l="${link_width}" w="${link4_length}" h="${link_width}" x_offset="${-link_width/2}" y_offset="${-link4_length/2}" z_offset="0.0" />
     </link>
-    <joint name="link4_joint" type="continuous">
+    <joint name="link4_joint" type="revolute">
       <origin xyz="${-link_width/2} ${-link5_length/2} 0.0" rpy="0 0.0 0.0"/>
       <parent link="link5"/>
       <child link="link4"/>
       <axis xyz="1 0 0.0"/>
+      <limit lower="-0.44" upper="1.74" effort="0.0" velocity="0.0"/>
     </joint>
   </xacro:macro>

Commit message: Add some code

File: src/car_description/urdf/five_link_car.urdf.xacro (robot description, xacro)
@@ -66,6 +66,16 @@
       <child link="link1"/>
       <axis xyz="1 0 0.0"/>
-      <limit lower="-1.74" upper="0.44" effort="0.0" velocity="0.0"/>
-    </joint>
+      <limit lower="-1.74" upper="0.44" effort="3.07" velocity="70"/>
+    </joint>
+    <transmission name="link1_joint_trans">
+      <type>transmission_interface/SimpleTransmission</type>
+      <joint name="link1_joint">
+        <hardwareInterface>hardware_interface/EffortJointInterface</hardwareInterface>
+      </joint>
+      <actuator name="link1_joint_motor">
+        <mechanicalReduction>1.0</mechanicalReduction>
+        <hardwareInterface>hardware_interface/EffortJointInterface</hardwareInterface>
+      </actuator>
+    </transmission>
     <link name="link2">
       <visual name="">
@@ -91,5 +101,5 @@
       <child link="link2"/>
       <axis xyz="1 0.0 0.0"/>
-      <limit lower="-0.4" upper="2.5" effort="0.0" velocity="0.0"/>
+      <limit lower="-0.4" upper="2.5" effort="3.07" velocity="70"/>
     </joint>
     <link name="link3">
@@ -116,5 +126,5 @@
       <child link="link3"/>
       <axis xyz="1 0.0 0.0"/>
-      <limit lower="-2.5" upper="0.4" effort="0.0" velocity="0.0"/>
+      <limit lower="-2.5" upper="0.4" effort="3.07" velocity="70"/>
     </joint>
     <link name="link4">
@@ -141,6 +151,16 @@
       <child link="link4"/>
       <axis xyz="1 0 0.0"/>
-      <limit lower="-0.44" upper="1.74" effort="0.0" velocity="0.0"/>
-    </joint>
+      <limit lower="-0.44" upper="1.74" effort="3.07" velocity="70"/>
+    </joint>
+    <transmission name="link4_joint_trans">
+      <type>transmission_interface/SimpleTransmission</type>
+      <joint name="link4_joint">
+        <hardwareInterface>hardware_interface/EffortJointInterface</hardwareInterface>
+      </joint>
+      <actuator name="link4_joint_motor">
+        <mechanicalReduction>1.0</mechanicalReduction>
+        <hardwareInterface>hardware_interface/EffortJointInterface</hardwareInterface>
+      </actuator>
+    </transmission>
   </xacro:macro>
   <xacro:property name="base_link_height" value="0.5" />
@@ -178,5 +198,5 @@
       </axis>
       <pose>0 ${link3_length} 0 0 0 0</pose>
-      <limit lower="-3.14" upper="3.14" effort="10" velocity="10"/>
+      <limit lower="-3.14" upper="3.14" effort="3.07" velocity="70"/>
     </joint>
   </gazebo>
